File: kicad/parasite.kicad_sch (KiCad schematic)
At the start: 29 parts, among them Q1 MMBT3906, Q4 Q_Photo_NPN, SW1 B3U-1000P, U1 E73-2G4M08S1C, U2 SHTC3, Y1 32.768kHz

Commit message: Javított nyák, más méretű optó tranzisztor (0806)
Parts:
- Q4: footprint snapeda:TR8 -> LED_SMD:LED_0805_2012Metric
Changed lines of the file:
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@@
       (effects (font (size 1.27 1.27)) (justify left))
     )
-    (property "Footprint" "snapeda:TR8" (at 215.9 120.65 0)
+    (property "Footprint" "LED_SMD:LED_0805_2012Metric" (at 215.9 120.65 0)
       (effects (font (size 1.27 1.27)) hide)
     )
